Commit message: update ar4.urdf.xacro with xacro files and macros for links, joints and materials

File: src/ar4_description/urdf/ar4.urdf.xacro (robot description, xacro)
@@ -1,202 +1,9 @@
 <?xml version="1.0"?>
 <robot name="my_robot" xmlns:xacro="http://www.ros.org/wiki/xacro">
-  <material name="grey">
-    <color rgba="0.79216 0.81961 0.93333 1" />
-  </material>
-  <link name="base_link">
-    <inertial>
-      <origin xyz="-0.041771 -1.1102E-16 0.033857" rpy="0 0 0" />
-      <mass value="1.407" />
-      <inertia ixx="0.0024719" ixy="-1.3675E-18" ixz="0.00018646"
-               iyy="0.00681"   iyz="1.095E-19"
-               izz="0.0070135" />
-    </inertial>
-    <visual>
-      <origin xyz="0 0 0" rpy="0 0 0" />
-      <geometry>
-        <mesh filename="package://ar4_description/meshes/visual/base_link.STL" />
-      </geometry>
-      <material name="grey" />
-    </visual>
-    <collision>
-      <origin xyz="0 0 0" rpy="0 0 0" />
-      <geometry>
-        <mesh filename="package://ar4_description/meshes/collision/base_link.STL" />
-      </geometry>
-    </collision>
-  </link>
-  <link name="1st_Link">
-    <inertial>
-      <origin xyz="0.0543 -0.020673 0.046417" rpy="0 0 0" />
-      <mass value="1.1495" />
-      <inertia ixx="0.0032387" ixy="0.00017789" ixz="-0.00039788"
-               iyy="0.0020161" iyz="0.00039611"
-               izz="0.0027855" />
-    </inertial>
-    <visual>
-      <origin xyz="0 0 0" rpy="0 0 0" />
-      <geometry>
-        <mesh filename="package://ar4_description/meshes/visual/1st_Link.STL" />
-      </geometry>
-      <material name="grey" />
-    </visual>
-    <collision>
-      <origin xyz="0 0 0" rpy="0 0 0" />
-      <geometry>
-        <mesh filename="package://ar4_description/meshes/collision/1st_Link.STL" />
-      </geometry>
-    </collision>
-  </link>
-  <joint name="Joint_0" type="revolute">
-    <origin xyz="0 0 0.0994" rpy="0 0 0" />
-    <parent link="base_link" />
-    <child link="1st_Link" />
-    <axis xyz="0 0 -1" />
-    <limit lower="-2.9671" upper="2.9671" effort="4" velocity="3.1" />
-  </joint>
-  <link name="2nd_Link">
-    <inertial>
-      <origin xyz="-1.5543E-15 -0.14784 -0.014918" rpy="0 0 0" />
-      <mass value="0.8363" />
-      <inertia ixx="0.008149"   ixy="9.6713E-18" ixz="-1.613E-18"
-               iyy="0.00093169" iyz="0.00089805"
-               izz="0.0076645" />
-    </inertial>
-    <visual>
-      <origin xyz="0 0 0" rpy="0 0 0" />
-      <geometry>
-        <mesh filename="package://ar4_description/meshes/visual/2nd_Link.STL" />
-      </geometry>
-      <material name="grey" />
-    </visual>
-    <collision>
-      <origin xyz="0 0 0" rpy="0 0 0" />
-      <geometry>
-        <mesh filename="package://ar4_description/meshes/collision/2nd_Link.STL" />
-      </geometry>
-    </collision>
-  </link>
-  <joint name="Joint_1" type="revolute">
-    <origin xyz="0.064201 0.064413 0.069869" rpy="-1.5708 0 0" />
-    <parent link="1st_Link" />
-    <child link="2nd_Link" />
-    <axis xyz="0 0 -1" />
-    <limit lower="-0.733" upper="1.5708" effort="57" velocity="0.63" />
-  </joint>
-  <link name="3rd_Link">
-    <inertial>
-      <origin xyz="0.0020169 0.017836 -0.07504" rpy="0 0 0" />
-      <mass value="0.27635" />
-      <inertia ixx="0.00030182" ixy="3.1988E-05" ixz="-5.1391E-06"
-               iyy="0.00023538" iyz="6.3261E-05"
-               izz="0.00031122" />
-    </inertial>
-    <visual>
-      <origin xyz="0 0 0" rpy="0 0 0" />
-      <geometry>
-        <mesh filename="package://ar4_description/meshes/visual/3rd_Link.STL" />
-      </geometry>
-      <material name="grey" />
-    </visual>
-    <collision>
-      <origin xyz="0 0 0" rpy="0 0 0" />
-      <geometry>
-        <mesh filename="package://ar4_description/meshes/collision/3rd_Link.STL" />
-      </geometry>
-    </collision>
-  </link>
-  <joint name="Joint_2" type="revolute">
-    <origin xyz="0 -0.305 0.016225" rpy="0 0 0" />
-    <parent link="2nd_Link" />
-    <child link="3rd_Link" />
-    <axis xyz="0 0 1" />
-    <limit lower="-1.5533" upper="0.9076" effort="20" velocity="0.63" />
-  </joint>
-  <link name="4th_Link">
-    <inertial>
-      <origin xyz="1.2523E-13 0.0044165 0.16589" rpy="0 0 0" />
-      <mass value="0.58728" />
-      <inertia ixx="0.0038961" ixy="6.9388E-13" ixz="-3.8354E-15"
-               iyy="0.0037675" iyz="-5.2921E-05"
-               izz="0.00034965" />
-    </inertial>
-    <visual>
-      <origin xyz="0 0 0" rpy="0 0 0" />
-      <geometry>
-        <mesh filename="package://ar4_description/meshes/visual/4th_Link.STL" />
-      </geometry>
-      <material name="grey" />
-    </visual>
-    <collision>
-      <origin xyz="0 0 0" rpy="0 0 0" />
-      <geometry>
-        <mesh filename="package://ar4_description/meshes/collision/4th_Link.STL" />
-      </geometry>
-    </collision>
-  </link>
-  <joint name="Joint_3" type="revolute">
-    <origin xyz="-0.078271 0 -0.090625" rpy="-1.5708 0 -1.5708" />
-    <parent link="3rd_Link" />
-    <child link="4th_Link" />
-    <axis xyz="0 0 -1" />
-    <limit lower="-2.8798" upper="2.8798" effort="1.6" velocity="2" />
-  </joint>
-  <link name="5th_Link">
-    <inertial>
-      <origin xyz="4.8184E-14 -0.01065 -0.040384" rpy="0 0 0" />
-      <mass value="0.13801" />
-      <inertia ixx="0.00010569" ixy="-5.0825E-17" ixz="1.6311E-16"
-               iyy="7.3011E-05" iyz="-7.9323E-06"
-               izz="6.2637E-05" />
-    </inertial>
-    <visual>
-      <origin xyz="0 0 0" rpy="0 0 0" />
-      <geometry>
-        <mesh filename="package://ar4_description/meshes/visual/5th_Link.STL" />
-      </geometry>
-      <material name="grey" />
-    </visual>
-    <collision>
-      <origin xyz="0 0 0" rpy="0 0 0" />
-      <geometry>
-        <mesh filename="package://ar4_description/meshes/collision/5th_Link.STL" />
-      </geometry>
-    </collision>
-  </link>
-  <joint name="Joint_4" type="revolute">
-    <origin xyz="0 -0.044813 0.29996" rpy="1.5708 0 0" />
-    <parent link="4th_Link" />
-    <child link="5th_Link" />
-    <axis xyz="0 0 -1" />
-    <limit lower="-1.8326" upper="1.8326" effort="81" velocity="0.16" />
-  </joint>
-  <link name="6th_Link">
-    <inertial>
-      <origin xyz="-2.2204E-16 0 -0.0070452" rpy="0 0 0" />
-      <mass value="0.015303" />
-      <inertia ixx="1.9052E-06" ixy="-1.4035E-19" ixz="-1.8528E-20"
-               iyy="1.4167E-06" iyz="9.3992E-21"
-               izz="2.619E-06" />
-    </inertial>
-    <visual>
-      <origin xyz="0 0 0" rpy="0 0 0" />
-      <geometry>
-        <mesh filename="package://ar4_description/meshes/visual/6th_Link.STL" />
-      </geometry>
-      <material name="grey" />
-    </visual>
-    <collision>
-      <origin xyz="0 0 0" rpy="0 0 0" />
-      <geometry>
-        <mesh filename="package://ar4_description/meshes/collision/6th_Link.STL" />
-      </geometry>
-    </collision>
-  </link>
-  <joint name="Joint_5" type="revolute">
-    <origin xyz="0 0.03625 -0.045781" rpy="1.5708 0 3.1416" />
-    <parent link="5th_Link" />
-    <child link="6th_Link" />
-    <axis xyz="0 0 1" />
-    <limit lower="-2.7053" upper="2.7053" effort="2.4" velocity="1.65" />
-  </joint>
+  <xacro:include filename="common_properties.xacro" />
+  <xacro:include filename="ar4.xacro" />
+  <!-- <xacro:include filename="my_robot_gazebo.xacro" />
+    <link name="world"/>
+   <xacro:joint_fixed name="world_fixed_joint" parent="world" child="base_link"
+    origin_xyz="0 0 0" origin_rpy="0 0 0" />  -->
 </robot>

Commit message: Adding ar4_moveit_config and run gazebo with ros2_control and moveit visualizing in Rviz

File: src/ar4_description/urdf/ar4.urdf.xacro (robot description, xacro)
@@ -1,11 +1,138 @@
 <?xml version="1.0"?>
-<robot name="my_robot" xmlns:xacro="http://www.ros.org/wiki/xacro">
+<robot name="AR4" xmlns:xacro="http://www.ros.org/wiki/xacro">
+  <!-- Import common properties and macros -->
   <xacro:include filename="common_properties.xacro" />
-  <xacro:include filename="ar4.xacro" />
-  <xacro:include filename="$(find ar4_description)/urdf/ar4_ros2_control.xacro"/>
-  <xacro:ar4_ros2_control use_mock_hardware="true"/>
-  <!-- <xacro:include filename="my_robot_gazebo.xacro" />
-    <link name="world"/>
-   <xacro:joint_fixed name="world_fixed_joint" parent="world" child="base_link"
-    origin_xyz="0 0 0" origin_rpy="0 0 0" />  -->
+  <!-- Import arm description -->
+  <xacro:include filename="arm.xacro" />
+  <!-- ═══════════════════════════════════════════════════════
+       ROS2_CONTROL — conditional on gazebo arg
+       ═══════════════════════════════════════════════════════ -->
+  <xacro:if value="$(arg gazebo)">
+    <!-- Gazebo physics hardware interface -->
+    <ros2_control name="GazeboSystem" type="system">
+      <hardware>
+        <plugin>gz_ros2_control/GazeboSimSystem</plugin>
+      </hardware>
+      <joint name="Joint_0">
+        <command_interface name="position">
+          <param name="min">-2.9671</param>
+          <param name="max">2.9671</param>
+        </command_interface>
+        <state_interface name="position"/>
+        <state_interface name="effort"/>
+      </joint>
+      <joint name="Joint_1">
+        <command_interface name="position">
+          <param name="min">-0.733</param>
+          <param name="max">1.5708</param>
+        </command_interface>
+        <state_interface name="position"/>
+        <state_interface name="effort"/>
+      </joint>
+      <joint name="Joint_2">
+        <command_interface name="position">
+          <param name="min">-1.5533</param>
+          <param name="max">0.9076</param>
+        </command_interface>
+        <state_interface name="position"/>
+        <state_interface name="effort"/>
+      </joint>
+      <joint name="Joint_3">
+        <command_interface name="position">
+          <param name="min">-2.8798</param>
+          <param name="max">2.8798</param>
+        </command_interface>
+        <state_interface name="position"/>
+        <state_interface name="effort"/>
+      </joint>
+      <joint name="Joint_4">
+        <command_interface name="position">
+          <param name="min">-1.8326</param>
+          <param name="max">1.8326</param>
+        </command_interface>
+        <state_interface name="position"/>
+        <state_interface name="effort"/>
+      </joint>
+      <joint name="Joint_5">
+        <command_interface name="position">
+          <param name="min">-2.7053</param>
+          <param name="max">2.7053</param>
+        </command_interface>
+        <state_interface name="position"/>
+        <state_interface name="effort"/>
+      </joint>
+    </ros2_control>
+    <!-- Gazebo plugin that loads gz_ros2_control -->
+    <gazebo>
+      <plugin
+          filename="gz_ros2_control-system"
+          name="gz_ros2_control::GazeboSimROS2ControlPlugin">
+        <parameters>$(find ar4_description)/config/controllers.yaml</parameters>
+      </plugin>
+    </gazebo>
+  </xacro:if>
+  <!-- ═══════════════════════════════════════════════════════
+       FAKE / MOCK hardware (no Gazebo)
+       ═══════════════════════════════════════════════════════ -->
+  <xacro:unless value="$(arg gazebo)">
+    <ros2_control name="Arm" type="system">
+      <hardware>
+        <plugin>mock_components/GenericSystem</plugin>
+      </hardware>
+      <joint name="Joint_0">
+        <command_interface name="position">
+          <param name="min">-2.9671</param>
+          <param name="max">2.9671</param>
+        </command_interface>
+        <state_interface name="position">
+          <param name="initial_value">0.0</param>
+        </state_interface>
+      </joint>
+      <joint name="Joint_1">
+        <command_interface name="position">
+          <param name="min">-0.733</param>
+          <param name="max">1.5708</param>
+        </command_interface>
+        <state_interface name="position">
+          <param name="initial_value">0.0</param>
+        </state_interface>
+      </joint>
+      <joint name="Joint_2">
+        <command_interface name="position">
+          <param name="min">-1.5533</param>
+          <param name="max">0.9076</param>
+        </command_interface>
+        <state_interface name="position">
+          <param name="initial_value">0.0</param>
+        </state_interface>
+      </joint>
+      <joint name="Joint_3">
+        <command_interface name="position">
+          <param name="min">-2.8798</param>
+          <param name="max">2.8798</param>
+        </command_interface>
+        <state_interface name="position">
+          <param name="initial_value">0.0</param>
+        </state_interface>
+      </joint>
+      <joint name="Joint_4">
+        <command_interface name="position">
+          <param name="min">-1.8326</param>
+          <param name="max">1.8326</param>
+        </command_interface>
+        <state_interface name="position">
+          <param name="initial_value">0.0</param>
+        </state_interface>
+      </joint>
+      <joint name="Joint_5">
+        <command_interface name="position">
+          <param name="min">-2.7053</param>
+          <param name="max">2.7053</param>
+        </command_interface>
+        <state_interface name="position">
+          <param name="initial_value">0.0</param>
+        </state_interface>
+      </joint>
+    </ros2_control>
+  </xacro:unless>
 </robot>

File: src/ar4_description/urdf/arm.xacro (robot description, xacro)
@@ -1,4 +1,16 @@
 <?xml version="1.0"?>
 <robot xmlns:xacro="http://www.ros.org/wiki/xacro">
+  <!-- ═══════════════════════════════════════════════════════
+       WORLD LINK + FIXED BASE
+       ═══════════════════════════════════════════════════════ -->
+  <link name="world"/>
+  <joint name="world_joint" type="fixed">
+    <origin xyz="0 0 0" rpy="0 0 ${PI/2}"/>
+    <parent link="world"/>
+    <child link="base_link"/>
+  </joint>
+  <!-- ═══════════════════════════════════════════════════════
+       LINKS
+       ═══════════════════════════════════════════════════════ -->
   <xacro:add_link name="base_link" mass="0.97407"
         inr_xyz="-0.039732 -9.8037E-07 0.023083" inr_rpy="0 0 0"
@@ -55,5 +67,5 @@
         inr_xyz="-0.011337 1.1704E-05 -0.040849" inr_rpy="0 0 0"
         vis_xyz="0 0 0" vis_rpy="0 0 0"
-        col_xyz="0 0 0" col_rpy="0 0 ${-pi/2.0}"
+        col_xyz="0 0 0" col_rpy="0 0 ${-PI/2.0}"
         ixx="2.3634E-05" ixy="3.2989E-09" ixz="-4.8512E-09"
         iyy="2.198E-05" iyz="7.5032E-09"
@@ -74,3 +86,9 @@
     axis_xyz="0 0 1" limit_lower="-2.7053" limit_upper="2.7053"
     limit_effort="2.4" limit_velocity="1.65" />
+    <link name="tool_link" />
+    <joint name="hand_tool_joint" type="fixed">
+        <parent link="6th_Link" />
+        <child link="tool_link" />
+        <origin xyz="0 0 0" rpy="0 0 0" />
+    </joint>
 </robot>

File: src/ar4_description/urdf/common_properties.xacro (robot description, xacro)
@@ -1,7 +1,17 @@
 <?xml version="1.0"?>
 <robot xmlns:xacro="http://www.ros.org/wiki/xacro">
+  <xacro:property name="PI" value="3.14159"/>
+  <xacro:property name="effort" value="30.0"/>
+  <xacro:property name="velocity" value="10.0"/>
+  <xacro:arg name="gazebo" default="true"/>
   <material name="grey">
     <color rgba="0.79216 0.81961 0.93333 1" />
   </material>
+  <material name="blue">
+    <color rgba="0 0 0.5 1" />
+  </material>
+  <!-- ═══════════════════════════════════════════════════════
+       MACROS
+       ═══════════════════════════════════════════════════════ -->
   <xacro:macro name="add_link" params="name mass
         inr_xyz inr_rpy vis_xyz vis_rpy col_xyz
@@ -40,10 +50,3 @@
     </joint>
   </xacro:macro>
-  <xacro:macro name="joint_fixed" params="name parent child origin_xyz origin_rpy">
-    <joint name="${name}" type="fixed">
-      <origin xyz="${origin_xyz}" rpy="${origin_rpy}" />
-      <parent link="${parent}" />
-      <child link="${child}" />
-    </joint>
-  </xacro:macro>
 </robot>

Commit message: Develop the main launch file for the 3 modes (Gazebo-Simulation, Mock-Component and Real-Hardware'still in progress')

File: src/ar4_description/urdf/ar4.urdf.xacro (robot description, xacro)
@@ -5,134 +5,13 @@
   <!-- Import arm description -->
   <xacro:include filename="arm.xacro" />
-  <!-- ═══════════════════════════════════════════════════════
-       ROS2_CONTROL — conditional on gazebo arg
-       ═══════════════════════════════════════════════════════ -->
-  <xacro:if value="$(arg gazebo)">
-    <!-- Gazebo physics hardware interface -->
-    <ros2_control name="GazeboSystem" type="system">
-      <hardware>
-        <plugin>gz_ros2_control/GazeboSimSystem</plugin>
-      </hardware>
-      <joint name="Joint_0">
-        <command_interface name="position">
-          <param name="min">-2.9671</param>
-          <param name="max">2.9671</param>
-        </command_interface>
-        <state_interface name="position"/>
-        <state_interface name="effort"/>
-      </joint>
-      <joint name="Joint_1">
-        <command_interface name="position">
-          <param name="min">-0.733</param>
-          <param name="max">1.5708</param>
-        </command_interface>
-        <state_interface name="position"/>
-        <state_interface name="effort"/>
-      </joint>
-      <joint name="Joint_2">
-        <command_interface name="position">
-          <param name="min">-1.5533</param>
-          <param name="max">0.9076</param>
-        </command_interface>
-        <state_interface name="position"/>
-        <state_interface name="effort"/>
-      </joint>
-      <joint name="Joint_3">
-        <command_interface name="position">
-          <param name="min">-2.8798</param>
-          <param name="max">2.8798</param>
-        </command_interface>
-        <state_interface name="position"/>
-        <state_interface name="effort"/>
-      </joint>
-      <joint name="Joint_4">
-        <command_interface name="position">
-          <param name="min">-1.8326</param>
-          <param name="max">1.8326</param>
-        </command_interface>
-        <state_interface name="position"/>
-        <state_interface name="effort"/>
-      </joint>
-      <joint name="Joint_5">
-        <command_interface name="position">
-          <param name="min">-2.7053</param>
-          <param name="max">2.7053</param>
-        </command_interface>
-        <state_interface name="position"/>
-        <state_interface name="effort"/>
-      </joint>
-    </ros2_control>
-    <!-- Gazebo plugin that loads gz_ros2_control -->
-    <gazebo>
-      <plugin
-          filename="gz_ros2_control-system"
-          name="gz_ros2_control::GazeboSimROS2ControlPlugin">
-        <parameters>$(find ar4_description)/config/controllers.yaml</parameters>
-      </plugin>
-    </gazebo>
-  </xacro:if>
-  <!-- ═══════════════════════════════════════════════════════
-       FAKE / MOCK hardware (no Gazebo)
-       ═══════════════════════════════════════════════════════ -->
-  <xacro:unless value="$(arg gazebo)">
-    <ros2_control name="Arm" type="system">
-      <hardware>
-        <plugin>mock_components/GenericSystem</plugin>
-      </hardware>
-      <joint name="Joint_0">
-        <command_interface name="position">
-          <param name="min">-2.9671</param>
-          <param name="max">2.9671</param>
-        </command_interface>
-        <state_interface name="position">
-          <param name="initial_value">0.0</param>
-        </state_interface>
-      </joint>
-      <joint name="Joint_1">
-        <command_interface name="position">
-          <param name="min">-0.733</param>
-          <param name="max">1.5708</param>
-        </command_interface>
-        <state_interface name="position">
-          <param name="initial_value">0.0</param>
-        </state_interface>
-      </joint>
-      <joint name="Joint_2">
-        <command_interface name="position">
-          <param name="min">-1.5533</param>
-          <param name="max">0.9076</param>
-        </command_interface>
-        <state_interface name="position">
-          <param name="initial_value">0.0</param>
-        </state_interface>
-      </joint>
-      <joint name="Joint_3">
-        <command_interface name="position">
-          <param name="min">-2.8798</param>
-          <param name="max">2.8798</param>
-        </command_interface>
-        <state_interface name="position">
-          <param name="initial_value">0.0</param>
-        </state_interface>
-      </joint>
-      <joint name="Joint_4">
-        <command_interface name="position">
-          <param name="min">-1.8326</param>
-          <param name="max">1.8326</param>
-        </command_interface>
-        <state_interface name="position">
-          <param name="initial_value">0.0</param>
-        </state_interface>
-      </joint>
-      <joint name="Joint_5">
-        <command_interface name="position">
-          <param name="min">-2.7053</param>
-          <param name="max">2.7053</param>
-        </command_interface>
-        <state_interface name="position">
-          <param name="initial_value">0.0</param>
-        </state_interface>
-      </joint>
-    </ros2_control>
-  </xacro:unless>
+  <gazebo>
+    <plugin
+        filename="gz_ros2_control-system"
+        name="gz_ros2_control::GazeboSimROS2ControlPlugin">
+      <parameters>$(find ar4_description)/config/controllers.yaml</parameters>
+    </plugin>
+  </gazebo>
+  <xacro:arg name="is_gazebo_sim" default="true"/>
+  <xacro:include filename="$(find ar4_description)/urdf/AR4.ros2_control.xacro" />
+  <xacro:arduinobot_ros2_control is_gazebo_sim="$(arg is_gazebo_sim)"/>
 </robot>
